File: kicad/cta.sch (KiCad schematic (older format))
At the start: 21 parts, among them Q1 2N3904, Q2 2N3906, U1 LM324

Commit message: Modified the warmup subcircuit
To initialize the circuit, a subcircuit was used that on powerup would
temporarily add voltage to the + leg of the op amp. Now this circuit adds
this voltage directly to the base of Q1. With this I could also remove
the resistor conecting both cricuits (Rs1).

I also decreased the fill zones tolerances and most of the board is now
filled.
Parts:
- removed Rs1: 220k, Resistor_THT:R_Axial_DIN0207_L6.3mm_D2.5mm_P10.16mm_Horizontal, symbol Device:R_US
Connections:
- wire segments 87 -> 88
Changed lines of the file:
@@
 EESchema Schematic File Version 4
+LIBS:cta-cache
 EELAYER 30 0
 EELAYER END
@@
 	5500 2400 5200 2400
 Wire Wire Line
-	5200 2400 5200 1850
+	5200 2400 5200 2300
 Wire Wire Line
 	2750 2050 2750 2500
@@
 Wire Wire Line
 	3300 2900 3600 2900
-$Comp
-L Device:R_US Rs1
-U 1 1 5F6C5636
-P 3600 2400
-F 0 "Rs1" V 3395 2400 50  0000 C CNN
-F 1 "220k" V 3486 2400 50  0000 C CNN
-F 2 "Resistor_THT:R_Axial_DIN0207_L6.3mm_D2.5mm_P10.16mm_Horizontal" V 3640 2390 50  0001 C CNN
-F 3 "~" H 3600 2400 50  0001 C CNN
-	1    3600 2400
-	-1   0    0    1
-$EndComp
 Wire Wire Line
 	5500 1650 5500 1600
@@
 $EndComp
 Wire Wire Line
-	3600 2850 3600 2550
-Connection ~ 3600 2850
-Wire Wire Line
-	3600 2250 3600 1950
-Wire Wire Line
 	5000 1100 5050 1100
 Wire Wire Line
@@
 	1    0    0    -1
 $EndComp
+Wire Wire Line
+	3600 1950 3600 2300
+Wire Wire Line
+	3600 2300 5200 2300
+Connection ~ 5200 2300
+Wire Wire Line
+	5200 2300 5200 1850
 $EndSCHEMATC

Commit message: Improved board layout and allowed for a power resistor.
Parts:
- added Ron1: 2k, Resistor_THT:R_Axial_DIN0207_L6.3mm_D2.5mm_P10.16mm_Horizontal, symbol Device:R_US
- Q1, Q2: footprint Package_TO_SOT_THT:TO-92_Inline -> Package_TO_SOT_THT:TO-92_Inline_Wide
- R2: footprint Resistor_THT:R_Axial_DIN0207_L6.3mm_D2.5mm_P10.16mm_Horizontal -> Resistor_THT:R_Axial_Power_L20.0mm_W6.4mm_P22.40mm
- Rtrans1: value 1k -> 2k
Connections:
- wire segments 88 -> 89
Changed lines of the file:
@@
 EESchema Schematic File Version 4
-LIBS:cta-cache
 EELAYER 30 0
 EELAYER END
@@
 F 0 "R2" H 3068 2696 50  0000 L CNN
 F 1 "15" H 3068 2605 50  0000 L CNN
-F 2 "Resistor_THT:R_Axial_DIN0207_L6.3mm_D2.5mm_P10.16mm_Horizontal" V 3040 2640 50  0001 C CNN
+F 2 "Resistor_THT:R_Axial_Power_L20.0mm_W6.4mm_P22.40mm" V 3040 2640 50  0001 C CNN
 F 3 "~" H 3000 2650 50  0001 C CNN
 	1    3000 2650
@@
 P 5500 2550
 F 0 "Rtrans1" H 5568 2596 50  0000 L CNN
-F 1 "1k" H 5568 2505 50  0000 L CNN
+F 1 "2k" H 5568 2505 50  0000 L CNN
 F 2 "Resistor_THT:R_Axial_DIN0207_L6.3mm_D2.5mm_P10.16mm_Horizontal" V 5540 2540 50  0001 C CNN
 F 3 "~" H 5500 2550 50  0001 C CNN
@@
 Wire Wire Line
 	5500 2400 5200 2400
-Wire Wire Line
-	5200 2400 5200 2300
 Wire Wire Line
 	2750 2050 2750 2500
@@
 F 0 "Q2" H 3891 1704 50  0000 L CNN
 F 1 "2N3906" H 3891 1795 50  0000 L CNN
-F 2 "Package_TO_SOT_THT:TO-92_Inline" H 3900 1675 50  0001 L CIN
+F 2 "Package_TO_SOT_THT:TO-92_Inline_Wide" H 3900 1675 50  0001 L CIN
 F 3 "https://www.fairchildsemi.com/datasheets/2N/2N3906.pdf" H 3700 1750 50  0001 L CNN
 	1    3700 1750
@@
 Wire Wire Line
 	5050 750  5050 1100
+Wire Wire Line
+	5150 3250 5400 3250
+Wire Wire Line
+	5400 3250 5400 3000
+Connection ~ 5400 3000
+Wire Wire Line
+	5400 3000 5500 3000
+Wire Wire Line
+	4850 3250 4550 3250
+Wire Wire Line
+	4550 3250 4550 3150
+Connection ~ 4550 3150
+Wire Wire Line
+	4550 3150 4750 3150
+$Comp
+L Transistor_BJT:2N3904 Q1
+U 1 1 5F7F4BD5
+P 5500 1850
+F 0 "Q1" H 5690 1896 50  0000 L CNN
+F 1 "2N3904" H 5690 1805 50  0000 L CNN
+F 2 "Package_TO_SOT_THT:TO-92_Inline_Wide" H 5700 1775 50  0001 L CIN
+F 3 "https://www.fairchildsemi.com/datasheets/2N/2N3904.pdf" H 5500 1850 50  0001 L CNN
+	1    5500 1850
+	1    0    0    -1
+$EndComp
 $Comp
 L Device:C C1
@@
 $EndComp
 Wire Wire Line
-	5150 3250 5400 3250
-Wire Wire Line
-	5400 3250 5400 3000
-Connection ~ 5400 3000
-Wire Wire Line
-	5400 3000 5500 3000
-Wire Wire Line
-	4850 3250 4550 3250
-Wire Wire Line
-	4550 3250 4550 3150
-Connection ~ 4550 3150
-Wire Wire Line
-	4550 3150 4750 3150
-$Comp
-L Transistor_BJT:2N3904 Q1
-U 1 1 5F7F4BD5
-P 5500 1850
-F 0 "Q1" H 5690 1896 50  0000 L CNN
-F 1 "2N3904" H 5690 1805 50  0000 L CNN
-F 2 "Package_TO_SOT_THT:TO-92_Inline" H 5700 1775 50  0001 L CIN
-F 3 "https://www.fairchildsemi.com/datasheets/2N/2N3904.pdf" H 5500 1850 50  0001 L CNN
-	1    5500 1850
-	1    0    0    -1
+	5200 1850 5200 2300
+$Comp
+L Device:R_US Ron1
+U 1 1 5F9763D1
+P 4250 2300
+F 0 "Ron1" V 4045 2300 50  0000 C CNN
+F 1 "2k" V 4136 2300 50  0000 C CNN
+F 2 "Resistor_THT:R_Axial_DIN0207_L6.3mm_D2.5mm_P10.16mm_Horizontal" V 4290 2290 50  0001 C CNN
+F 3 "~" H 4250 2300 50  0001 C CNN
+	1    4250 2300
+	0    1    1    0
 $EndComp
 Wire Wire Line
 	3600 1950 3600 2300
 Wire Wire Line
-	3600 2300 5200 2300
+	3600 2300 4100 2300
+Wire Wire Line
+	4400 2300 5200 2300
 Connection ~ 5200 2300
 Wire Wire Line
-	5200 2300 5200 1850
+	5200 2300 5200 2400
 $EndSCHEMATC

Commit message: Removed a terminal block and increased the power termninal block to 3
The circuit uses the same ground for power and signal. So I removed the signal terminal block and added another terminal to the power terminal block
Parts:
- removed VOUT1: VOUT, TerminalBlock:TerminalBlock_bornier-2_P5.08mm, symbol Connector:Conn_01x02_Male
- VALIM1: footprint TerminalBlock:TerminalBlock_bornier-2_P5.08mm -> TerminalBlock:TerminalBlock_bornier-3_P5.08mm; symbol Connector:Conn_01x02_Male -> Connector_Generic:Conn_01x03
Connections:
- wire segments 89 -> 95
Changed lines of the file:
@@
 Wire Wire Line
 	2750 2500 3000 2500
-$Comp
-L Connector:Conn_01x02_Male VALIM1
-U 1 1 5F6BC983
-P 5600 1300
-F 0 "VALIM1" V 5662 1344 50  0000 L CNN
-F 1 "Vcc" V 5753 1344 50  0000 L CNN
-F 2 "TerminalBlock:TerminalBlock_bornier-2_P5.08mm" H 5600 1300 50  0001 C CNN
-F 3 "~" H 5600 1300 50  0001 C CNN
-	1    5600 1300
-	0    1    1    0
-$EndComp
 Wire Wire Line
 	2750 3300 2750 4050
@@
 Wire Wire Line
 	5500 1500 5300 1500
-Connection ~ 5500 1500
 Wire Wire Line
 	6150 4300 5300 4300
@@
 Wire Wire Line
 	5400 3600 6150 3600
-$Comp
-L Connector:Conn_01x02_Male VOUT1
-U 1 1 5F6FF1B4
-P 7700 4050
-F 0 "VOUT1" H 7672 3932 50  0000 R CNN
-F 1 "VOUT" H 7672 4023 50  0000 R CNN
-F 2 "TerminalBlock:TerminalBlock_bornier-2_P5.08mm" H 7700 4050 50  0001 C CNN
-F 3 "~" H 7700 4050 50  0001 C CNN
-	1    7700 4050
-	-1   0    0    1
-$EndComp
 Wire Wire Line
 	7200 3950 7500 3950
 Connection ~ 7200 3950
-Wire Wire Line
-	7500 4050 7500 4300
-Wire Wire Line
-	7500 4300 6150 4300
-Connection ~ 6150 4300
 Connection ~ 6000 3200
 Wire Wire Line
 	6000 3200 6000 4050
 Wire Wire Line
-	5500 1100 5300 1100
+	5500 1100 5450 1100
 Wire Wire Line
 	5300 1100 5300 1500
@@
 $EndComp
 Wire Wire Line
-	5850 1150 6000 1150
-Wire Wire Line
-	6000 1150 6000 1500
+	6000 1150 6000 1250
 Wire Wire Line
 	6300 2600 6300 1100
@@
 Wire Wire Line
 	5200 2300 5200 2400
+$Comp
+L Connector_Generic:Conn_01x03 VALIM1
+U 1 1 5F6BC983
+P 5550 1350
+F 0 "VALIM1" V 5612 1394 50  0000 L CNN
+F 1 "Vcc" V 5703 1394 50  0000 L CNN
+F 2 "TerminalBlock:TerminalBlock_bornier-3_P5.08mm" H 5550 1350 50  0001 C CNN
+F 3 "~" H 5550 1350 50  0001 C CNN
+	1    5550 1350
+	0    1    1    0
+$EndComp
+Wire Wire Line
+	5450 1150 5450 1100
+Connection ~ 5450 1100
+Wire Wire Line
+	5450 1100 5300 1100
+Wire Wire Line
+	5550 1150 5550 1250
+Wire Wire Line
+	5550 1250 6000 1250
+Connection ~ 6000 1250
+Wire Wire Line
+	6000 1250 6000 1500
+Wire Wire Line
+	5850 1150 6000 1150
+Wire Wire Line
+	7500 3950 7500 800
+Wire Wire Line
+	7500 800  5650 800
+Wire Wire Line
+	5650 800  5650 1150
 $EndSCHEMATC

Commit message: Set new values for components
One of the things I noticed with the circuit is an asymmetry when increasing wind speed vs decreasing. When increasing, the response is fast. But when decreasing it is very low.

This is to be expected: the electronics respond much faster than the cooling: the maximum colling rate happens when there is no current and therefore heat transfer within the thermistor is the slow part.

To make response more symmetric, I increased the the resistors at the op amp input from 1k to 47k. This introduced a new problem: the capacitor would not charge fast enough for the initial charge subcircuit. I could increase the capacitoor in this subcircuit and increase the resistance as well. I haven't tested these solutions. What I did was increase the feedback capacitance from 100nF to 1uF. The circuit is working and the response is much more symmetric.

Another change was decreasing the base resistors. They are not necessary. I still left a low resistor just to keep the layout. But they could be replaced by wires (that's what I tested). This improves response time (which doesn't really matter).
Parts:
- C1: value C -> 1u
- R1: value 150 -> 100
- R2: value 15 -> 10
- R3: value 1.5k -> 1k
- Rfa1, Rfb1: value 1k -> 47k
- Ron1, Rtrans1: value 2k -> 10
- Roo0: value R_US -> 10
Changed lines of the file:
@@
 P 2500 2650
 F 0 "R1" H 2568 2696 50  0000 L CNN
-F 1 "150" H 2568 2605 50  0000 L CNN
+F 1 "100" H 2568 2605 50  0000 L CNN
 F 2 "Resistor_THT:R_Axial_DIN0207_L6.3mm_D2.5mm_P10.16mm_Horizontal" V 2540 2640 50  0001 C CNN
 F 3 "~" H 2500 2650 50  0001 C CNN
@@
 P 3000 2650
 F 0 "R2" H 3068 2696 50  0000 L CNN
-F 1 "15" H 3068 2605 50  0000 L CNN
+F 1 "10" H 3068 2605 50  0000 L CNN
 F 2 "Resistor_THT:R_Axial_Power_L20.0mm_W6.4mm_P22.40mm" V 3040 2640 50  0001 C CNN
 F 3 "~" H 3000 2650 50  0001 C CNN
@@
 P 2500 3150
 F 0 "R3" H 2568 3196 50  0000 L CNN
-F 1 "1.5k" H 2568 3105 50  0000 L CNN
+F 1 "1k" H 2568 3105 50  0000 L CNN
 F 2 "Resistor_THT:R_Axial_DIN0207_L6.3mm_D2.5mm_P10.16mm_Horizontal" V 2540 3140 50  0001 C CNN
 F 3 "~" H 2500 3150 50  0001 C CNN
@@
 P 3750 2850
 F 0 "Rfa1" V 3545 2850 50  0000 C CNN
-F 1 "1k" V 3636 2850 50  0000 C CNN
+F 1 "47k" V 3636 2850 50  0000 C CNN
 F 2 "Resistor_THT:R_Axial_DIN0207_L6.3mm_D2.5mm_P10.16mm_Horizontal" V 3790 2840 50  0001 C CNN
 F 3 "~" H 3750 2850 50  0001 C CNN
@@
 P 3750 3150
 F 0 "Rfb1" V 3545 3150 50  0000 C CNN
-F 1 "1k" V 3636 3150 50  0000 C CNN
+F 1 "47k" V 3636 3150 50  0000 C CNN
 F 2 "Resistor_THT:R_Axial_DIN0207_L6.3mm_D2.5mm_P10.16mm_Horizontal" V 3790 3140 50  0001 C CNN
 F 3 "~" H 3750 3150 50  0001 C CNN
@@
 P 5500 2550
 F 0 "Rtrans1" H 5568 2596 50  0000 L CNN
-F 1 "2k" H 5568 2505 50  0000 L CNN
+F 1 "10" H 5568 2505 50  0000 L CNN
 F 2 "Resistor_THT:R_Axial_DIN0207_L6.3mm_D2.5mm_P10.16mm_Horizontal" V 5540 2540 50  0001 C CNN
 F 3 "~" H 5500 2550 50  0001 C CNN
@@
 P 4050 1600
 F 0 "Roo0" H 4118 1646 50  0000 L CNN
-F 1 "R_US" H 4118 1555 50  0000 L CNN
+F 1 "10" H 4118 1555 50  0000 L CNN
 F 2 "Resistor_THT:R_Axial_DIN0207_L6.3mm_D2.5mm_P10.16mm_Horizontal" V 4090 1590 50  0001 C CNN
 F 3 "~" H 4050 1600 50  0001 C CNN
@@
 P 5000 3250
 F 0 "C1" V 4748 3250 50  0000 C CNN
-F 1 "C" V 4839 3250 50  0000 C CNN
+F 1 "1u" V 4839 3250 50  0000 C CNN
 F 2 "Capacitor_THT:C_Rect_L7.2mm_W4.5mm_P5.00mm_FKS2_FKP2_MKS2_MKP2" H 5038 3100 50  0001 C CNN
 F 3 "~" H 5000 3250 50  0001 C CNN
@@
 P 4250 2300
 F 0 "Ron1" V 4045 2300 50  0000 C CNN
-F 1 "2k" V 4136 2300 50  0000 C CNN
+F 1 "10" V 4136 2300 50  0000 C CNN
 F 2 "Resistor_THT:R_Axial_DIN0207_L6.3mm_D2.5mm_P10.16mm_Horizontal" V 4290 2290 50  0001 C CNN
 F 3 "~" H 4250 2300 50  0001 C CNN

Commit message: Replaced transistor KSP2222A for BC517
The BC517 is a darlington transistor and the response of the anemometer is much faster (when increasing wind speed). Why would I care about that if I went to all the trouble to make the response more symmetric?

It really depends on the objective. If I want to measure the mean speed in a turbulent flow, using the more symmetric response is better. But If I want to estimate wind gusts, the faster response time could do that! This change inm transistor really has no downsides.
Parts:
- Q1: value 2N3904 -> BC517; symbol Transistor_BJT:2N3904 -> Transistor_BJT:BC517
Changed lines of the file:
@@
 	4550 3150 4750 3150
 $Comp
-L Transistor_BJT:2N3904 Q1
+L Transistor_BJT:BC517 Q1
 U 1 1 5F7F4BD5
 P 5500 1850
 F 0 "Q1" H 5690 1896 50  0000 L CNN
-F 1 "2N3904" H 5690 1805 50  0000 L CNN
+F 1 "BC517" H 5690 1805 50  0000 L CNN
 F 2 "Package_TO_SOT_THT:TO-92_Inline_Wide" H 5700 1775 50  0001 L CIN
 F 3 "https://www.fairchildsemi.com/datasheets/2N/2N3904.pdf" H 5500 1850 50  0001 L CNN

Commit message: I found out the trouble: too much power dissipated on the tranistor
During normal operation, the current is low and therefore the voltage at the top of the bridge is low and the transistor needs to reduce a lot of voltage and dissipate a lot of heat. After normal operation for a little time the transistor would burn up.

I see 2 solutions:
 1. Replace the transistor
 2. Modify the resistors

I think I will do #2 anyway and do #2.
Parts:
- added D1: 1N4148, Diode_THT:D_DO-35_SOD27_P7.62mm_Horizontal, symbol Diode:1N4148
- Ron1: value 10 -> 47k
Connections:
- net +24V: now also D1.2 (A); no longer Q2.1 (E)
- new net: D1.1 (K), Q2.1 (E)
Changed lines of the file:
@@
 	5800 1500 5600 1500
-Wire Wire Line
-	3600 1550 3600 750
 Wire Wire Line
 	3600 750  5050 750
@@
 P 4250 2300
 F 0 "Ron1" V 4045 2300 50  0000 C CNN
-F 1 "10" V 4136 2300 50  0000 C CNN
+F 1 "47k" V 4136 2300 50  0000 C CNN
 F 2 "Resistor_THT:R_Axial_DIN0207_L6.3mm_D2.5mm_P10.16mm_Horizontal" V 4290 2290 50  0001 C CNN
 F 3 "~" H 4250 2300 50  0001 C CNN
@@
 Wire Wire Line
 	5650 800  5650 1150
+$Comp
+L Diode:1N4148 D1
+U 1 1 5F9D38B7
+P 3600 1200
+F 0 "D1" V 3646 1120 50  0000 R CNN
+F 1 "1N4148" V 3555 1120 50  0000 R CNN
+F 2 "Diode_THT:D_DO-35_SOD27_P7.62mm_Horizontal" H 3600 1025 50  0001 C CNN
+F 3 "https://assets.nexperia.com/documents/data-sheet/1N4148_1N4448.pdf" H 3600 1200 50  0001 C CNN
+	1    3600 1200
+	0    -1   -1   0
+$EndComp
+Wire Wire Line
+	3600 1050 3600 750
+Wire Wire Line
+	3600 1550 3600 1350
 $EndSCHEMATC

Commit message: Replaced the transistor from BC517 to TIP120 and resistors on the bridge
The resistors on the top of the bridge now have the same value as on the bottom of the bridge. This decreased the power dissipated in the transistor.

The new transistor can also include a heat sink dependeing on application. The setup is working on the protoboard. I has been working for the last hour, voltage input can be decreased to 15V and the system will still start. At 13V it takes a while, perhaps a larger capacitor for startup procedure will help.
Parts:
- Q1: value BC517 -> TIP122; footprint Package_TO_SOT_THT:TO-92_Inline_Wide -> Package_TO_SOT_THT:TO-220-3_Vertical; symbol Transistor_BJT:BC517 -> Transistor_BJT:TIP122
Connections:
- net +24V: now also Q1.2 (C); no longer Q1.1 (C)
- net at Ron1.1, Rtrans1.1: now also Q1.1 (B); no longer Q1.2 (B)
Changed lines of the file:
@@
 	4550 3150 4750 3150
-$Comp
-L Transistor_BJT:BC517 Q1
-U 1 1 5F7F4BD5
-P 5500 1850
-F 0 "Q1" H 5690 1896 50  0000 L CNN
-F 1 "BC517" H 5690 1805 50  0000 L CNN
-F 2 "Package_TO_SOT_THT:TO-92_Inline_Wide" H 5700 1775 50  0001 L CIN
-F 3 "https://www.fairchildsemi.com/datasheets/2N/2N3904.pdf" H 5500 1850 50  0001 L CNN
-	1    5500 1850
-	1    0    0    -1
-$EndComp
 $Comp
 L Device:C C1
@@
 Wire Wire Line
 	3600 1550 3600 1350
+$Comp
+L Transistor_BJT:TIP122 Q1
+U 1 1 5F7F4BD5
+P 5500 1850
+F 0 "Q1" H 5690 1896 50  0000 L CNN
+F 1 "TIP122" H 5690 1805 50  0000 L CNN
+F 2 "Package_TO_SOT_THT:TO-220-3_Vertical" H 5700 1775 50  0001 L CIN
+F 3 "https://www.fairchildsemi.com/datasheets/2N/2N3904.pdf" H 5500 1850 50  0001 L CNN
+	1    5500 1850
+	1    0    0    -1
+$EndComp
 $EndSCHEMATC

Commit message: Cleaned up the schematics
The circuit is much clearer! I have tested the circuit 24 hours and it is working. Now I have to test it on a wind tunnel and checkout how well it operates.
Parts:
- Q1: value TIP122 -> TIP120; symbol Transistor_BJT:TIP122 -> Transistor_BJT:TIP120
- Q2: value 2N3906 -> KSP2907
- Ron1: value 47k -> 10
- Roo1: value R_US -> 100k
- Roo2: value R_US -> 12k
- Rw1: value Conn_01x02_Male -> Conn
Connections:
- net VOUTPUT: now reaches U1.8, U1.9 (-), VALIM1.1 (Pin_1)
- net +24V renamed VCC
- net GNDPWR renamed GND
Other:
- note added: "Circuit for turning on the Q1 transistor"
- note added: "Output voltage divider and follower\n"
- moved on the sheet: Coo1, D1, Q1, Q2, Ron1, Roo0, Roo1, Roo2, Rtrans1, U1E, VALIM1
