File: kicad/cta.sch (KiCad schematic (older format))
At the start: 21 parts, among them Q1 TIP120, Q2 KSP2907, U1 LM324

Commit message: Used the last op amp to implement an active low pass output filter
I think this is the best strategy to get a symmetric behavior when heating or cooling. Just get a time constant larger than the corresponding cooling time constant.
Parts:
- added Cf2: 10u, Capacitor_THT:CP_Radial_D5.0mm_P2.50mm, symbol Device:CP
- added Rf2: 10k, Resistor_THT:R_Axial_DIN0207_L6.3mm_D2.5mm_P10.16mm_Horizontal, symbol Device:R_US
- added unit 4 of U1
- U1: footprint Package_DIP:DIP-14_W7.62mm -> Package_DIP:DIP-14_W7.62mm_LongPads
Connections:
- net GND: now also Cf2.2
- net VOUTPUT: now also U1.13 (-), U1.14; no longer U1.8, U1.9 (-)
- new net: Rf2.2, U1.8, U1.9 (-)
- new net: Cf2.1, Rf2.1, U1.12 (+)
Changed lines of the file:
@@
 F 0 "U1" H 5050 3367 50  0000 C CNN
 F 1 "LM324" H 5050 3276 50  0000 C CNN
-F 2 "Package_DIP:DIP-14_W7.62mm" H 5000 3100 50  0001 C CNN
+F 2 "Package_DIP:DIP-14_W7.62mm_LongPads" H 5000 3100 50  0001 C CNN
 F 3 "http://www.ti.com/lit/ds/symlink/lm2902-n.pdf" H 5100 3200 50  0001 C CNN
 	1    5050 3000
@@
 F 0 "U1" H 5050 3967 50  0000 C CNN
 F 1 "LM324" H 5050 3876 50  0000 C CNN
-F 2 "Package_DIP:DIP-14_W7.62mm" H 5000 3700 50  0001 C CNN
+F 2 "Package_DIP:DIP-14_W7.62mm_LongPads" H 5000 3700 50  0001 C CNN
 F 3 "http://www.ti.com/lit/ds/symlink/lm2902-n.pdf" H 5100 3800 50  0001 C CNN
 	2    5050 3600
@@
 F 0 "U1" H 6900 4317 50  0000 C CNN
 F 1 "LM324" H 6900 4226 50  0000 C CNN
-F 2 "Package_DIP:DIP-14_W7.62mm" H 6850 4050 50  0001 C CNN
+F 2 "Package_DIP:DIP-14_W7.62mm_LongPads" H 6850 4050 50  0001 C CNN
 F 3 "http://www.ti.com/lit/ds/symlink/lm2902-n.pdf" H 6950 4150 50  0001 C CNN
 	3    6900 3950
@@
 F 0 "U1" H 3708 4446 50  0000 L CNN
 F 1 "LM324" H 3708 4355 50  0000 L CNN
-F 2 "Package_DIP:DIP-14_W7.62mm" H 3700 4500 50  0001 C CNN
+F 2 "Package_DIP:DIP-14_W7.62mm_LongPads" H 3700 4500 50  0001 C CNN
 F 3 "http://www.ti.com/lit/ds/symlink/lm2902-n.pdf" H 3800 4600 50  0001 C CNN
 	5    3750 4400
@@
 Wire Wire Line
 	5500 2150 5500 3000
-Text Label 7500 3950 0    50   ~ 0
+Text Label 9100 4050 0    50   ~ 0
 VOUTPUT
 Text Label 2450 1150 0    50   ~ 0
@@
 Text Notes 5400 4750 0    79   ~ 0
 Output voltage divider and follower\n
+$Comp
+L Amplifier_Operational:LM324 U1
+U 4 1 5FA2AA8D
+P 8500 4050
+F 0 "U1" H 8500 4417 50  0000 C CNN
+F 1 "LM324" H 8500 4326 50  0000 C CNN
+F 2 "Package_DIP:DIP-14_W7.62mm_LongPads" H 8450 4150 50  0001 C CNN
+F 3 "http://www.ti.com/lit/ds/symlink/lm2902-n.pdf" H 8550 4250 50  0001 C CNN
+	4    8500 4050
+	1    0    0    -1
+$EndComp
+$Comp
+L Device:R_US Rf2
+U 1 1 5FA2D98F
+P 7650 3950
+F 0 "Rf2" H 7718 3996 50  0000 L CNN
+F 1 "10k" H 7718 3905 50  0000 L CNN
+F 2 "Resistor_THT:R_Axial_DIN0207_L6.3mm_D2.5mm_P10.16mm_Horizontal" V 7690 3940 50  0001 C CNN
+F 3 "~" H 7650 3950 50  0001 C CNN
+	1    7650 3950
+	0    1    1    0
+$EndComp
+Wire Wire Line
+	7800 3950 7900 3950
+$Comp
+L Device:CP Cf2
+U 1 1 5FA3187E
+P 7900 4100
+F 0 "Cf2" H 8018 4146 50  0000 L CNN
+F 1 "10u" H 8018 4055 50  0000 L CNN
+F 2 "Capacitor_THT:CP_Radial_D5.0mm_P2.50mm" H 7938 3950 50  0001 C CNN
+F 3 "~" H 7900 4100 50  0001 C CNN
+	1    7900 4100
+	1    0    0    -1
+$EndComp
+Connection ~ 7900 3950
+Wire Wire Line
+	7900 3950 8200 3950
+$Comp
+L power:GND #PWR0113
+U 1 1 5FA340D0
+P 7900 4250
+F 0 "#PWR0113" H 7900 4000 50  0001 C CNN
+F 1 "GND" H 7905 4077 50  0000 C CNN
+F 2 "" H 7900 4250 50  0001 C CNN
+F 3 "" H 7900 4250 50  0001 C CNN
+	1    7900 4250
+	1    0    0    -1
+$EndComp
+Wire Wire Line
+	8800 4050 8950 4050
+Wire Wire Line
+	8950 4050 8950 4300
+Wire Wire Line
+	8950 4300 8200 4300
+Wire Wire Line
+	8200 4300 8200 4150
+Connection ~ 8950 4050
+Wire Wire Line
+	8950 4050 9100 4050
 $EndSCHEMATC

Commit message: The circuit was not working with low noise, low offset op amp
I removed the input filter and the cicrcuit works with precision op amps. Stilll need to test the circuit exhaustively.
Parts:
- C1: value 1u -> 0.15u
- Cf1: value 1u -> 0
- Rfa1, Rfb1: value 47k -> 1
- Ron1, Rtrans1: value 10 -> 1
Changed lines of the file:
@@
 P 3750 2850
 F 0 "Rfa1" V 3545 2850 50  0000 C CNN
-F 1 "47k" V 3636 2850 50  0000 C CNN
+F 1 "1" V 3636 2850 50  0000 C CNN
 F 2 "Resistor_THT:R_Axial_DIN0207_L6.3mm_D2.5mm_P10.16mm_Horizontal" V 3790 2840 50  0001 C CNN
 F 3 "~" H 3750 2850 50  0001 C CNN
@@
 P 3750 3150
 F 0 "Rfb1" V 3545 3150 50  0000 C CNN
-F 1 "47k" V 3636 3150 50  0000 C CNN
+F 1 "1" V 3636 3150 50  0000 C CNN
 F 2 "Resistor_THT:R_Axial_DIN0207_L6.3mm_D2.5mm_P10.16mm_Horizontal" V 3790 3140 50  0001 C CNN
 F 3 "~" H 3750 3150 50  0001 C CNN
@@
 P 4100 3000
 F 0 "Cf1" H 4215 3046 50  0000 L CNN
-F 1 "1u" H 4215 2955 50  0000 L CNN
+F 1 "0" H 4215 2955 50  0000 L CNN
 F 2 "Capacitor_THT:C_Rect_L7.2mm_W4.5mm_P5.00mm_FKS2_FKP2_MKS2_MKP2" H 4138 2850 50  0001 C CNN
 F 3 "~" H 4100 3000 50  0001 C CNN
@@
 P 5000 3250
 F 0 "C1" V 4748 3250 50  0000 C CNN
-F 1 "1u" V 4839 3250 50  0000 C CNN
+F 1 "0.15u" V 4839 3250 50  0000 C CNN
 F 2 "Capacitor_THT:C_Rect_L7.2mm_W4.5mm_P5.00mm_FKS2_FKP2_MKS2_MKP2" H 5038 3100 50  0001 C CNN
 F 3 "~" H 5000 3250 50  0001 C CNN
@@
 P 4050 2150
 F 0 "Rtrans1" H 4118 2196 50  0000 L CNN
-F 1 "10" H 4118 2105 50  0000 L CNN
+F 1 "1" H 4118 2105 50  0000 L CNN
 F 2 "Resistor_THT:R_Axial_DIN0207_L6.3mm_D2.5mm_P10.16mm_Horizontal" V 4090 2140 50  0001 C CNN
 F 3 "~" H 4050 2150 50  0001 C CNN
@@
 P 4650 1900
 F 0 "Ron1" V 4445 1900 50  0000 C CNN
-F 1 "10" V 4536 1900 50  0000 C CNN
+F 1 "1" V 4536 1900 50  0000 C CNN
 F 2 "Resistor_THT:R_Axial_DIN0207_L6.3mm_D2.5mm_P10.16mm_Horizontal" V 4690 1890 50  0001 C CNN
 F 3 "~" H 4650 1900 50  0001 C CNN
